Commit message: Add collision to ingenuity and perseverance

File: ingenuity/ingenuity.urdf (robot description, URDF)
Before this commit: robot , 13 links, 12 joints
Links:
- link Body_MHS_BottomBlades_v16: geometry collision mesh filename=./meshes/MHS_BottomBlades_v16.glb scale=1 1 1; visual mesh filename=./meshes/MHS_BottomBlades_v16.glb scale=1 1 1
- link Body_MHS_Leg01_v16: geometry collision mesh filename=./meshes/MHS_Leg01_v16.glb scale=1 1 1; visual mesh filename=./meshes/MHS_Leg01_v16.glb scale=1 1 1
- link Body_MHS_Leg02_v16: geometry collision mesh filename=./meshes/MHS_Leg02_v16.glb scale=1 1 1; visual mesh filename=./meshes/MHS_Leg02_v16.glb scale=1 1 1
- link Body_MHS_Leg03_v16: geometry collision mesh filename=./meshes/MHS_Leg03_v16.glb scale=1 1 1; visual mesh filename=./meshes/MHS_Leg03_v16.glb scale=1 1 1
- link Body_MHS_Leg04_v16: geometry collision mesh filename=./meshes/MHS_Leg04_v16.glb scale=1 1 1; visual mesh filename=./meshes/MHS_Leg04_v16.glb scale=1 1 1
- link Body_MHS_MainBody_v16: geometry collision mesh filename=./meshes/MHS_MainBody_v16.glb scale=1 1 1; visual mesh filename=./meshes/MHS_MainBody_v16.glb scale=1 1 1
- link Body_MHS_TopBlades_v16: geometry collision mesh filename=./meshes/MHS_TopBlades_v16.glb scale=1 1 1; visual mesh filename=./meshes/MHS_TopBlades_v16.glb scale=1 1 1

File: perseverance/perseverance.urdf (robot description, URDF)
Before this commit: robot Perseverance, 115 links, 114 joints
Links:
- link Body_Chassis: geometry collision mesh filename=./meshes/CHASSIS.gltf scale=1 1 1; visual mesh filename=./meshes/CHASSIS.gltf scale=1 1 1
- link Body_RA_Link1: geometry collision mesh filename=./meshes/Arm_LINK_1.gltf scale=1 1 1; visual mesh filename=./meshes/Arm_LINK_1.gltf scale=1 1 1
- link Body_RA_Link2: geometry collision mesh filename=./meshes/Arm_LINK_2.gltf scale=1 1 1; visual mesh filename=./meshes/Arm_LINK_2.gltf scale=1 1 1
- link Body_RA_Link3: geometry collision mesh filename=./meshes/Arm_LINK_3.gltf scale=1 1 1; visual mesh filename=./meshes/Arm_LINK_3.gltf scale=1 1 1
- link Body_RA_Link4: geometry collision mesh filename=./meshes/Arm_LINK_4.gltf scale=1 1 1; visual mesh filename=./meshes/Arm_LINK_4.gltf scale=1 1 1
- link Body_RA_Link5: geometry collision mesh filename=./meshes/Arm_LINK_5.gltf scale=1 1 1; visual mesh filename=./meshes/Arm_LINK_5.gltf scale=1 1 1
- link Body_WheelLeftFront: geometry collision mesh filename=./meshes/Wheel_LeftFront.gltf scale=1 1 1; visual mesh filename=./meshes/Wheel_LeftFront.gltf scale=1 1 1
- link Body_WheelLeftMiddle: geometry collision mesh filename=./meshes/Wheel_LeftMiddle.gltf scale=1 1 1; visual mesh filename=./meshes/Wheel_LeftMiddle.gltf scale=1 1 1
- link Body_WheelLeftRear: geometry collision mesh filename=./meshes/Wheel_LeftRear.gltf scale=1 1 1; visual mesh filename=./meshes/Wheel_LeftRear.gltf scale=1 1 1
- link Body_WheelRightFront: geometry collision mesh filename=./meshes/Wheel_RightFront.gltf scale=1 1 1; visual mesh filename=./meshes/Wheel_RightFront.gltf scale=1 1 1
- link Body_WheelRightMiddle: geometry collision mesh filename=./meshes/Wheel_RightMiddle.gltf scale=1 1 1; visual mesh filename=./meshes/Wheel_RightMiddle.gltf scale=1 1 1
- link Body_WheelRightRear: geometry collision mesh filename=./meshes/Wheel_RightRear.gltf scale=1 1 1; visual mesh filename=./meshes/Wheel_RightRear.gltf scale=1 1 1
