Commit message: Update perseverance.urdf with inertial tags removed

File: perseverance/perseverance.urdf (robot description, URDF)
Before this commit: robot Perseverance, 115 links, 114 joints
Links:
- removed link Frame_STEER_LF
- added link _LF
- link Body_BogieLeft: mass 1 -> None
- link Body_BogieRight: mass 1 -> None
- link Body_Chassis: mass 900 -> None
- link Body_CorerFeed: mass 1 -> None
- link Body_Differential: mass 1 -> None
- link Body_HGA_AZ: mass 1 -> None
- link Body_HGA_EL: mass 1 -> None
- link Body_MHS_DebrisShield: mass 1 -> None
- link Body_RA_Base: mass 1 -> None
- link Body_RA_Link1: mass 1 -> None
- link Body_RA_Link2: mass 1 -> None
- link Body_RA_Link3: mass 1 -> None
- link Body_RA_Link4: mass 1 -> None
- link Body_RA_Link5: mass 1 -> None
- link Body_RSM_AZ: mass 1 -> None
- link Body_RSM_EL: mass 1 -> None
- link Body_RockerLeft: mass 1 -> None
- link Body_RockerRight: mass 1 -> None
- link Body_SHERLOC_Cap: mass 1 -> None
- link Body_StabilizerFar: mass 1 -> None
- link Body_StabilizerNear: mass 1 -> None
- link Body_SteerLeftFront: mass 1 -> None
- link Body_SteerLeftRear: mass 1 -> None
- link Body_SteerRightFront: mass 1 -> None
- link Body_SteerRightRear: mass 1 -> None
- link Body_Turret: mass 1 -> None
- link Body_WATSON_Cap: mass 1 -> None
- link Body_WheelLeftFront: mass 1 -> None
- link Body_WheelLeftMiddle: mass 1 -> None
- link Body_WheelLeftRear: mass 1 -> None
- link Body_WheelRightFront: mass 1 -> None
- link Body_WheelRightMiddle: mass 1 -> None
- link Body_WheelRightRear: mass 1 -> None
- link Frame_ANT: mass 1 -> None
- link Frame_ATS1: mass 1 -> None
- link Frame_ATS2: mass 1 -> None
- link Frame_ATS3: mass 1 -> None
- link Frame_ATS4: mass 1 -> None
- link Frame_ATS5: mass 1 -> None
- link Frame_BOGIE_L: mass 1 -> None
- link Frame_BOGIE_R: mass 1 -> None
- link Frame_CAL_MC1: mass 1 -> None
- link Frame_CAL_MC2: mass 1 -> None
- link Frame_CAL_PIXL: mass 1 -> None
- link Frame_CAL_SC: mass 1 -> None
- link Frame_CAL_SHERLOC: mass 1 -> None
- link Frame_DIFF: mass 1 -> None
- link Frame_DOCKING_POST: mass 1 -> None
- link Frame_DRILL: mass 1 -> None
- link Frame_FCS: mass 1 -> None
- link Frame_FHC1: mass 1 -> None
- link Frame_FHC1_FOV: mass 1 -> None
- link Frame_FHC2: mass 1 -> None
- link Frame_FHC2_FOV: mass 1 -> None
- link Frame_FHC3: mass 1 -> None
- link Frame_FHC3_FOV: mass 1 -> None
- link Frame_FHC4: mass 1 -> None
- link Frame_FHC4_FOV: mass 1 -> None
- link Frame_FHCB: mass 1 -> None
- link Frame_GDRT: mass 1 -> None
- link Frame_HGAG: mass 1 -> None
- link Frame_HGAS: mass 1 -> None
- link Frame_HS: mass 1 -> None
- link Frame_ICU: mass 1 -> None
- link Frame_MAZ: mass 1 -> None
- link Frame_MCL: mass 1 -> None
- link Frame_MCR: mass 1 -> None
- link Frame_MEL: mass 1 -> None
- link Frame_MI: mass 1 -> None
- link Frame_MOXIE: mass 1 -> None
- link Frame_NCL: mass 1 -> None
- link Frame_NCL_FOV: mass 1 -> None
- link Frame_NCR: mass 1 -> None
- link Frame_NCR_FOV: mass 1 -> None
- link Frame_PIXL: mass 1 -> None
- link Frame_RA1: mass 1 -> None
- link Frame_RA2: mass 1 -> None
- link Frame_RA3: mass 1 -> None
- link Frame_RA4: mass 1 -> None
- link Frame_RA5: mass 1 -> None
- link Frame_RA6: mass 1 -> None
- link Frame_RA_BASE: mass 1 -> None
- link Frame_RDS: mass 1 -> None
- link Frame_RHC1: mass 1 -> None
- link Frame_RHC1_FOV: mass 1 -> None
- link Frame_RHC2: mass 1 -> None
- link Frame_RHC2_FOV: mass 1 -> None
- link Frame_RIMFAX: mass 1 -> None
- link Frame_RIMUA: mass 1 -> None
- link Frame_RIMUB: mass 1 -> None
- link Frame_RMECH: mass 1 -> None
- link Frame_RNAV: mass 1 -> None
- link Frame_ROCKER_L: mass 1 -> None
- link Frame_ROCKER_R: mass 1 -> None
- link Frame_SCI: mass 1 -> None
- link Frame_SCIR: mass 1 -> None
- link Frame_SCLIBS: mass 1 -> None
- link Frame_SCRMI: mass 1 -> None
- link Frame_SHERLOC: mass 1 -> None
- link Frame_STEER_LR: mass 1 -> None
- link Frame_STEER_RF: mass 1 -> None
- link Frame_STEER_RR: mass 1 -> None
- link Frame_TIRS: mass 1 -> None
- link Frame_TURRET: mass 1 -> None
- link Frame_WATSON: mass 1 -> None
- link Frame_WHEEL_LF: mass 1 -> None
- link Frame_WHEEL_LM: mass 1 -> None
- link Frame_WHEEL_LR: mass 1 -> None
- link Frame_WHEEL_RF: mass 1 -> None
- link Frame_WHEEL_RM: mass 1 -> None
- link Frame_WHEEL_RR: mass 1 -> None
- link Frame_WS1: mass 1 -> None
- link Frame_WS2: mass 1 -> None
- link ground: mass 0 -> None
Joints:
- removed joint Joint_for_Frame_STEER_RF
- removed joint Joint_for_Frame_STEER_RR
- added joint Joint_for__RF: type fixed, parent Body_SteerRightFront, child _RF, origin xyz=0 0 0 rpy=0 -0 0
- added joint Joint_for__RR: type fixed, parent Body_SteerRightRear, child _RR, origin xyz=0 0 0 rpy=0 -0 0
- joint Joint_for_Frame_STEER_LR: child Frame_STEER_LR -> _LR
